File: Main Board/MoritzKlein-ADSR.kicad_sch (KiCad schematic)
At the start: 34 parts, among them J1 Gate, J2 Out, J3 Conn_01x06, J4 Conn_01x06, U1 TL074

Commit message: Upload Schematics
Other:
- note added: "Power"
- title: (none) -> KOSMO - Moritz Klein - ADSR
- moved on the sheet: C1, C2, C3, C4, C5, C6, C7, C8, D1, D2, D3, D4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
